File: schemas/kicad/main_board/main_board.kicad_pcb (KiCad board)
At the start: 2 copper layers, 91 parts

Commit message: From now on login with ssh
Parts:
- C_3V3A1, C_ENGINE_TEMP_SENSE_P1000: footprint Capacitor_THT:C_Disc_D3.0mm_W1.6mm_P2.50mm -> Capacitor_THT:C_Disc_D4.3mm_W1.9mm_P5.00mm
- Q_BAT_REV_CONN1, Q_TEMP_SENSORS_REF1: moved to B.Cu
- Q_BAT_SW_CONN1: renamed from Q_BAT_REV_CONN2; moved to B.Cu
- R_ENGINE_TEMP_SENSE1, R_ENGINE_TEMP_SENSE_OPAMP1: footprint Resistor_THT:R_Axial_DIN0204_L3.6mm_D1.6mm_P5.08mm_Horizontal -> Resistor_THT:R_Axial_DIN0204_L3.6mm_D1.6mm_P7.62mm_Horizontal
- R_ENGINE_TEMP_SENSE_OPAMP4, R_EXT_TEMP_SENSE_OPAMP4: footprint Resistor_THT:R_Axial_DIN0204_L3.6mm_D1.6mm_P5.08mm_Horizontal -> Resistor_THT:R_Axial_DIN0204_L3.6mm_D1.6mm_P2.54mm_Vertical
- U_ENGINE_TEMP_SENSE_OP_AMP1: footprint Package_DIP:DIP-14_W7.62mm -> Package_DIP:DIP-14_W7.62mm_LongPads
- moved C_ENGINE_TEMP_SENSE_P1000 240.8 mm to (238.8, 196.8), turned to 270 degrees
- moved J_ENGINE_TEMP_P1000_IN1 229.0 mm to (234.9, 218.4), turned to 270 degrees
- moved C_TEMP_SENSOR_REF1 225.4 mm to (245.1, 133.3), turned to 270 degrees
- moved R_ENGINE_TEMP_SENSE_DIV1 219.2 mm to (234.9, 205.7), turned to 270 degrees
- moved R_TEMP_SENSOR2 217.3 mm to (236.2, 147.3)
- moved Q_TEMP_SENSOR_REF2 204.1 mm to (231.1, 149.9), turned to 90 degrees
- moved R_TEMP_SENSOR1 199.8 mm to (231.1, 137.2), turned to 270 degrees
- moved R_ENGINE_TEMP_SENSE1 189.0 mm to (228.6, 186.7), turned to 180 degrees
- moved R_ENGINE_TEMP_SENSE_OPAMP2 184.6 mm to (231.1, 200.7), turned to 90 degrees
- moved R_ENGINE_TEMP_SENSE_OPAMP3 183.3 mm to (226.1, 196.8)
- moved RV_ENGINE_TEMP_SENSE_TRIM_POT1 177.8 mm to (210.8, 186.7), turned to 180 degrees
- moved R_ENGINE_TEMP_SENSE_OPAMP4 173.7 mm to (226.1, 207.0)
- moved U_VREF_TEMP_SENSORS1 168.3 mm to (222.2, 144.8), turned to 90 degrees
- moved U_ENGINE_TEMP_SENSE_OP_AMP1 168.3 mm to (212.1, 194.3)
- moved C_TEMP_SENSOR_REF2 166.7 mm to (241.3, 147.3), turned to 270 degrees
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Routing:
- net GND: track 0.00 -> 148.6 mm
- net TEMP_SENSOR_3V_SUP: track 0.00 -> 68.8 mm
- net 3V3A: track 0.00 -> 48.2 mm
- net -BATT: track 0.00 -> 47.2 mm
- net Net-(R_ENGINE_TEMP_SENSE_OPAMP1-Pad1): track 0.00 -> 19.1 mm
- net +3V3: track 0.00 -> 19.1 mm
- net Net-(C_TEMP_SENSOR_REF2-Pad1): track 0.00 -> 18.8 mm
- net Net-(C_ENGINE_TEMP_SENSE_P1000-Pad2): track 0.00 -> 18.2 mm
- net Net-(Q_BAT_SW_CONN1-Pad1): track 0.00 -> 17.7 mm
- net BAT+_AFTER_MAIN_DRIVE: track 0.00 -> 17.2 mm
- net Net-(R_ENGINE_TEMP_SENSE_OPAMP2-Pad1): track 0.00 -> 14.8 mm
- net Net-(RV_ENGINE_TEMP_SENSE_TRIM_POT1-Pad2): track 0.00 -> 14.7 mm
- net +BATT: track 0.00 -> 14.3 mm
- net Net-(R_BAT_SENSORS_REF2-Pad1): track 0.00 -> 13.2 mm
- net Net-(Q_TEMP_SENSORS_REF1-Pad1): track 0.00 -> 12.9 mm
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Other:
- net class Default: clearance 0.2 -> 0.4; trace_width 0.25 -> 0.3
- net class Power added: clearance 0.8, trace_width 0.3, via_dia 0.8, via_drill 0.4
- rule trace_clearance: 0.2 -> 0.4
