File: schemas/kicad/main_board/main_board.sch (KiCad schematic (older format))
At the start: 87 parts

Commit message: Initial board file was created. NUCLEO board symbol was removed, and now there are female pin connectors in place of it. For simplicity reasons, and because of wrong footprint included in this lib.
Parts:
- removed U_CONTROL_BOARD1: NUCLEO64-F103RB, Module:ST_Morpho_Connector_144_STLink, symbol MY_MCU_MODULE:NUCLEO64-F103RB
- added J_STM_ADC1, J_STM_VCC1: Conn_01x03_Female, Connector_PinSocket_2.54mm:PinSocket_1x03_P2.54mm_Vertical, symbol Connector:Conn_01x03_Female
- added J_STM_COM1: Conn_01x09_Female, Connector_PinSocket_2.54mm:PinSocket_1x09_P2.54mm_Vertical, symbol Connector:Conn_01x09_Female
- added J_STM_GND1: Conn_01x06_Female, Connector_PinSocket_2.54mm:PinSocket_1x06_P2.54mm_Vertical, symbol Connector:Conn_01x06_Female
- added J_STM_OUT_SIG1: Conn_01x04_Female, Connector_PinSocket_2.54mm:PinSocket_1x04_P2.54mm_Vertical, symbol Connector:Conn_01x04_Female
- C_3V3A1, C_3V3A2, C_BAT_BRIDGE_DECAP1, C_EXT_TEMP_DECAP1: footprint (none) -> Capacitor_THT:C_Disc_D3.0mm_W1.6mm_P2.50mm
- C_BAT_BRIDGE_DECAP2: renamed from C_BAT_BRIDGE_DECAP1; footprint (none) -> Capacitor_THT:C_Disc_D3.0mm_W1.6mm_P2.50mm
- C_ENGINE_TEMP_SENSE_DECAP1: renamed from C_ENGINE_TEMP_SENSE_DECAP; footprint (none) -> Capacitor_THT:C_Disc_D3.0mm_W1.6mm_P2.50mm
- C_EXT_TEMP_DECAP2: renamed from C_EXT_TEMP_DECAP; footprint (none) -> Capacitor_THT:C_Disc_D3.0mm_W1.6mm_P2.50mm
- FB1: renamed from FB?; footprint (none) -> Resistor_THT:R_Axial_DIN0204_L3.6mm_D1.6mm_P5.08mm_Horizontal
- R_3V3A1: renamed from R_3V3A; footprint (none) -> Resistor_THT:R_Axial_DIN0204_L3.6mm_D1.6mm_P5.08mm_Horizontal
- U_BT1: renamed from U_BT; footprint (none) -> Connector_PinHeader_2.54mm:PinHeader_1x06_P2.54mm_Vertical
- renumbered C_3V3_IN to C_3V3_IN1, Q_BAT_REV_CONN2 to Q_BAT_SW_CONN1, R_MAIN_DRIVE_G_UP to R_MAIN_DRIVE_G_UP1
Connections:
- net +3V3: now also J_STM_VCC1.2 (Pin_2)
- net 3V3A: now also J_STM_VCC1.1 (Pin_1)
- net BAT_V_BRIDGE_OUT: now also J_STM_ADC1.1 (Pin_1)
- net BT_RXD: now also J_STM_COM1.2 (Pin_2)
- net BT_STATE: now also J_STM_COM1.1 (Pin_1)
- net BT_TXD: now also J_STM_COM1.3 (Pin_3)
- net ENGINE_TEMP_SENSOR_OUT: now also J_STM_ADC1.3 (Pin_3)
- net EXT_TEMP_SENSOR_OUT: now also J_STM_ADC1.2 (Pin_2)
- net EXT_TEMP_SENSOR_SEL_A: now also J_STM_OUT_SIG1.3 (Pin_3)
- net EXT_TEMP_SENSOR_SEL_B: now also J_STM_OUT_SIG1.4 (Pin_4)
- net GND: now also J_STM_GND1.1 (Pin_1), J_STM_GND1.2 (Pin_2), J_STM_GND1.3 (Pin_3), J_STM_GND1.4 (Pin_4), J_STM_GND1.5 (Pin_5), J_STM_GND1.6 (Pin_6), J_STM_VCC1.3 (Pin_3)
- net IMU_CS: now also J_STM_COM1.4 (Pin_4)
- net IMU_INT1: now also J_STM_COM1.9 (Pin_9)
- net IMU_INT2: now also J_STM_COM1.8 (Pin_8)
- net IMU_SCL: now also J_STM_COM1.7 (Pin_7)
- net IMU_SDI: now also J_STM_COM1.5 (Pin_5)
- net IMU_SDO: now also J_STM_COM1.6 (Pin_6)
- net OFF_SIG: now also J_STM_OUT_SIG1.2 (Pin_2)
- net TEMP_SENSOR_3V_SUP: no longer C_EXT_TEMP_SENSE_P1.2, C_EXT_TEMP_SENSE_P2.2, C_EXT_TEMP_SENSE_P3.2, J_EXT_TEMP_P1000_IN1.1 (Pin_1), J_EXT_TEMP_P1000_IN2.1 (Pin_1), J_EXT_TEMP_P1000_IN3.1 (Pin_1), R_EXT_TEMP_SENSE_DIV1.2, R_EXT_TEMP_SENSE_DIV2.2, R_EXT_TEMP_SENSE_DIV3.2, U_EXT_TEMP_SENSE_MUX1.12 (X0), U_EXT_TEMP_SENSE_MUX1.14 (X1), U_EXT_TEMP_SENSE_MUX1.15 (X2)
- net TEMP_SENSOR_REF_ON_SIG: now also J_STM_OUT_SIG1.1 (Pin_1)
- net BT_EN: no longer names the net of U_BT1.6 (EN)
- new net: C_EXT_TEMP_SENSE_P1.2, J_EXT_TEMP_P1000_IN1.1 (Pin_1), R_EXT_TEMP_SENSE_DIV1.2, U_EXT_TEMP_SENSE_MUX1.12 (X0)
- new net: C_EXT_TEMP_SENSE_P2.2, J_EXT_TEMP_P1000_IN2.1 (Pin_1), R_EXT_TEMP_SENSE_DIV2.2, U_EXT_TEMP_SENSE_MUX1.14 (X1)
- new net: C_EXT_TEMP_SENSE_P3.2, J_EXT_TEMP_P1000_IN3.1 (Pin_1), R_EXT_TEMP_SENSE_DIV3.2, U_EXT_TEMP_SENSE_MUX1.15 (X2)
- no-connect marks 15 -> 2
Other:
- note added: "BT CONNECTOR"
- note added: "STM CONNECTOR"
- moved on the sheet: C_STM_A_DECAP2, C_STM_DECAP1

Commit message: From now on login with ssh
Parts:
- C_3V3A1: footprint Capacitor_THT:C_Disc_D3.0mm_W1.6mm_P2.50mm -> Capacitor_THT:C_Disc_D4.3mm_W1.9mm_P5.00mm
Changed lines of the file:
@@
 F 0 "C_3V3A1" H 3040 1646 50  0000 L CNN
 F 1 "1u" H 3040 1555 50  0000 L CNN
-F 2 "Capacitor_THT:C_Disc_D3.0mm_W1.6mm_P2.50mm" H 2963 1450 50  0001 C CNN
+F 2 "Capacitor_THT:C_Disc_D4.3mm_W1.9mm_P5.00mm" H 2963 1450 50  0001 C CNN
 F 3 "~" H 2925 1600 50  0001 C CNN
 	1    2925 1600
